File: PCB/STM32SENSEHAT/power.kicad_sch (KiCad schematic)
At the start: 32 parts, among them IC1 DW01A, J1 USB_B_Micro, J7 Conn_01x05_Pin, Q1 NMOS, Q2 NMOS, U1 MCP1700x-330xxTT, U2 TP4056, U3 FT230XQ

Commit message: rework of top level sheet, MCU, power and sensor sheet
Parts:
- removed R7, R8: R_Small, symbol Device:R_Small
- C10, C11: value C_Small -> 1uF
- C7, C8: value C_Small -> 10uF
- C9: value C_Small -> 0.1uF
- R10: value R_Small -> 1k
- R4: value R_Small -> 0.4R
- R5: value R_Small -> 1k0
- R6: value R_Small -> 10k
- R9: value R_Small -> 100R
Connections:
- net GND: no longer U2.1 (TEMP)
- net !CHRG: no longer names the net of D2.1 (K), U2.7 (~{CHRG})
- net !STDBY: no longer names the net of D1.1 (K), U2.6 (~{STDBY})
- net BAT renamed BT_P
- net RXD renamed UART_TX
- net TXD renamed UART_RX
- no-connect marks 2 -> 3
Other:
- note added: "BATTERY CHARGER"
- note added: "BATTERY MANAGMENT SYSTEM"
- note added: "BATTERY PROTECTION"
- note added: "I/O INTERFACE"
- note added: "USB-FTDI INTERFACE"
- note added: "VOLTAGE REGULATOR"
- company: (none) -> IMPERIUM
- title: (none) -> POWER MANAGEMENT MODULE
- moved on the sheet: BT1, C1, C10, C11, C2, C3, C4, C5, C6, C7, C8, C9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
