File: PCB/STM32SENSEHAT/STM32SENSEHAT.kicad_pcb (KiCad board)
At the start: 2 copper layers, 100 x 100 mm, 83 parts, among them J1 USB_B_Micro, J10 Conn_01x01_Pin, J11 Conn_01x02_Pin, J2 Conn_01x05_Pin, J5 Conn_01x24_Pin, J8 Conn_01x24_Pin, J9 Conn_01x10_Pin, Q1 FS8205A, SW1 SW_Push, U1 MCP1700x-330xxTT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

Commit message: Added Justin's Feedback
Parts:
- added J3: USB_B_Micro, footprints:USB_Conn_JLC_LCSC_C404969, F.Cu at (199.6, 58.0)
- added R22: 1k0, Resistor_SMD:R_0805_2012Metric, F.Cu at (116.4, 61.8)
Connections:
- D5 pad 2: Net-(D4-A) -> Net-(D5-A)
- U9 pad 3: /MCU MODULE/USB_DN -> Net-(J3-D-)
- U9 pad 4: /MCU MODULE/USB_DP -> Net-(J3-D+)
Routing:
- net /MCU MODULE/USB_DN: track 157.2 -> 72.9 mm
- net /MCU MODULE/USB_DP: track 127.0 -> 46.6 mm
- net 5VUSB: track 248.6 -> 287.7 mm
- net Net-(J3-D-): track 0.00 -> 27.0 mm
- net Net-(J3-D+): track 0.00 -> 26.3 mm
- net Net-(D4-A): track 20.7 -> 5.98 mm
- net Net-(D5-A): track 0.00 -> 7.27 mm
