File: PCB/STM32SENSEHAT/mcu.kicad_sch (KiCad schematic)
At the start: 34 parts, among them J1 USB_B_Micro, J5 Conn_01x24_Pin, J6 Conn_01x10_Pin, J7 Conn_01x05_Pin, J8 Conn_01x24_Pin, SW1 SW_Push, U6 CAT24C256, U9 FT234XD-R, U9 STLINK_UCT, X1 XXDCELNANF-8MHZ

Commit message: Added Justin's Feedback
Parts:
- added J1: USB_B_Micro, footprints:USB_Conn_JLC_LCSC_C404969, symbol Connector:USB_B_Micro
Connections:
- net +5V: now also J1.1 (VBUS)
- net GND: now also J1.4 (ID), J1.5 (GND), J1.6 (Shield)
- net USB_DN: no longer U9.3 (USB_DM)
- net USB_DP: no longer U9.4 (USB_DP)
- new net: J1.2 (D-), U9.3 (USB_DM)
- new net: J1.3 (D+), U9.4 (USB_DP)
Changed lines of the file:
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@@
   (junction (at 36.83 171.45) (diameter 0) (color 0 0 0 0)
   )
+  (junction (at 67.31 88.9) (diameter 0) (color 0 0 0 0)
+  )
+  (junction (at 68.58 88.9) (diameter 0) (color 0 0 0 0)
+  )
   (junction (at 257.81 48.26) (diameter 0) (color 0 0 0 0)
   )
@@
     (stroke (width 0) (type default))
   )
+  (wire (pts (xy 78.74 78.74) (xy 76.2 78.74))
+    (stroke (width 0) (type default))
+  )
   (wire (pts (xy 91.44 219.71) (xy 100.33 219.71))
     (stroke (width 0) (type default))
@@
     (stroke (width 0) (type default))
   )
+  (wire (pts (xy 78.74 76.2) (xy 78.74 78.74))
+    (stroke (width 0) (type default))
+  )
+  (wire (pts (xy 76.2 76.2) (xy 77.47 76.2))
+    (stroke (width 0) (type default))
+  )
   (wire (pts (xy 283.21 44.45) (xy 283.21 48.26))
     (stroke (width 0) (type default))
@@
     (stroke (width 0) (type default))
   )
-  (wire (pts (xy 90.17 68.58) (xy 90.17 69.85))
+  (wire (pts (xy 90.17 63.5) (xy 90.17 69.85))
     (stroke (width 0) (type default))
   )
@@
     (stroke (width 0) (type default))
   )
+  (wire (pts (xy 76.2 81.28) (xy 76.2 88.9))
+    (stroke (width 0) (type default))
+  )
   (wire (pts (xy 274.32 86.36) (xy 266.7 86.36))
     (stroke (width 0) (type default))
@@
     (stroke (width 0) (type default))
   )
+  (wire (pts (xy 66.04 88.9) (xy 67.31 88.9))
+    (stroke (width 0) (type default))
+  )
   (wire (pts (xy 95.25 153.67) (xy 95.25 175.26))
     (stroke (width 0) (type default))
@@
     (stroke (width 0) (type default))
   )
+  (wire (pts (xy 78.74 71.12) (xy 78.74 63.5))
+    (stroke (width 0) (type default))
+  )
   (wire (pts (xy 208.28 93.98) (xy 213.36 93.98))
     (stroke (width 0) (type default))
@@
     (stroke (width 0) (type default))
   )
+  (wire (pts (xy 76.2 88.9) (xy 68.58 88.9))
+    (stroke (width 0) (type default))
+  )
   (wire (pts (xy 351.79 186.69) (xy 359.41 186.69))
     (stroke (width 0) (type default))
@@
     (stroke (width 0) (type default))
   )
+  (wire (pts (xy 78.74 63.5) (xy 90.17 63.5))
+    (stroke (width 0) (type default))
+  )
   (wire (pts (xy 227.33 171.45) (xy 233.68 171.45))
     (stroke (width 0) (type default))
@@
     (stroke (width 0) (type default))
   )
-  (wire (pts (xy 88.9 68.58) (xy 90.17 68.58))
-    (stroke (width 0) (type default))
-  )
   (wire (pts (xy 68.58 158.75) (xy 71.12 158.75))
     (stroke (width 0) (type default))
@@
     (stroke (width 0) (type default))
   )
+  (wire (pts (xy 76.2 71.12) (xy 78.74 71.12))
+    (stroke (width 0) (type default))
+  )
   (wire (pts (xy 227.33 217.17) (xy 233.68 217.17))
     (stroke (width 0) (type default))
@@
     (stroke (width 0) (type default))
   )
-  (wire (pts (xy 81.28 76.2) (xy 90.17 76.2))
+  (wire (pts (xy 78.74 76.2) (xy 90.17 76.2))
     (stroke (width 0) (type default))
   )
@@
     (stroke (width 0) (type default))
   )
+  (wire (pts (xy 68.58 88.9) (xy 67.31 88.9))
+    (stroke (width 0) (type default))
+  )
+  (wire (pts (xy 81.28 77.47) (xy 77.47 77.47))
+    (stroke (width 0) (type default))
+  )
   (wire (pts (xy 208.28 76.2) (xy 213.36 76.2))
     (stroke (width 0) (type default))
@@
     (stroke (width 0) (type default))
   )
+  (wire (pts (xy 68.58 86.36) (xy 68.58 88.9))
+    (stroke (width 0) (type default))
+  )
+  (wire (pts (xy 81.28 78.74) (xy 81.28 77.47))
+    (stroke (width 0) (type default))
+  )
+  (wire (pts (xy 77.47 77.47) (xy 77.47 76.2))
+    (stroke (width 0) (type default))
+  )
   (wire (pts (xy 49.53 170.18) (xy 49.53 176.53))
     (stroke (width 0) (type default))
@@
     (stroke (width 0) (type default))
   )
+  (wire (pts (xy 66.04 86.36) (xy 66.04 88.9))
+    (stroke (width 0) (type default))
+  )
   (wire (pts (xy 57.15 161.29) (xy 71.12 161.29))
     (stroke (width 0) (type default))
@@
     (fill (type none))
   )
-  (rectangle (start 68.58 21.59) (end 138.43 99.06)
+  (rectangle (start 53.34 21.59) (end 138.43 99.06)
     (stroke (width 1) (type default))
     (fill (type none))
@@
     (effects (font (size 1.27 1.27)) (justify left bottom))
   )
-  (label "USB_DN" (at 81.28 76.2 0) (fields_autoplaced)
-    (effects (font (size 1.27 1.27)) (justify left bottom))
-  )
   (label "PA10" (at 264.16 209.55 0) (fields_autoplaced)
     (effects (font (size 1.27 1.27)) (justify left bottom))
@@
     (effects (font (size 1.27 1.27)) (justify left bottom))
   )
-  (label "USB_DP" (at 81.28 78.74 0) (fields_autoplaced)
-    (effects (font (size 1.27 1.27)) (justify left bottom))
-  )
   (label "VBUS" (at 100.33 209.55 0) (fields_autoplaced)
     (effects (font (size 1.27 1.27)) (justify left bottom))
@@
     )
   )
-  (global_label "5VUSB" (shape input) (at 88.9 68.58 180) (fields_autoplaced)
-    (effects (font (size 1.27 1.27)) (justify right))
-    (property "Intersheetrefs" "${INTERSHEET_REFS}" (at 79.8861 68.58 0)
-      (effects (font (size 1.27 1.27)) (justify right) hide)
+  (global_label "5VUSB" (shape input) (at 83.82 63.5 90) (fields_autoplaced)
+    (effects (font (size 1.27 1.27)) (justify left))
+    (property "Intersheetrefs" "${INTERSHEET_REFS}" (at 83.82 54.4861 90)
+      (effects (font (size 1.27 1.27)) (justify left) hide)
     )
   )
@@
     )
   )
+  (symbol (lib_id "Connector:USB_B_Micro") (at 68.58 76.2 0) (unit 1)
+    (in_bom yes) (on_board yes) (dnp no) (fields_autoplaced)
+    (property "Reference" "J1" (at 68.58 64.77 0)
+      (effects (font (size 1.27 1.27)))
+    )
+    (property "Value" "USB_B_Micro" (at 68.58 67.31 0)
+      (effects (font (size 1.27 1.27)))
+    )
+    (property "Footprint" "footprints:USB_Conn_JLC_LCSC_C404969" (at 72.39 77.47 0)
+      (effects (font (size 1.27 1.27)) hide)
+    )
+    (property "Datasheet" "~" (at 72.39 77.47 0)
+      (effects (font (size 1.27 1.27)) hide)
+    )
+    (property "Basic" "" (at 68.58 76.2 0)
+      (effects (font (size 1.27 1.27)) hide)
+    )
+    (property "DNP" "" (at 68.58 76.2 0)
+      (effects (font (size 1.27 1.27)) hide)
+    )
+    (property "Extended" "" (at 68.58 76.2 0)
+      (effects (font (size 1.27 1.27)) hide)
+    )
+    (property "MOQ and Attrition" "" (at 68.58 76.2 0)
+      (effects (font (size 1.27 1.27)) hide)
+    )
+    (property "Price" "" (at 68.58 76.2 0)
+      (effects (font (size 1.27 1.27)) hide)
+    )
+    (pin "1")
+    (pin "2")
+    (pin "3")
+    (pin "4")
+    (pin "5")
+    (pin "6")
+    (instances
+      (project "mcu"
+        (path "/b04b5b28-ecb7-486f-a400-248cc160a7e5"
+          (reference "J1") (unit 1)
+        )
+      )
+      (project "STM32SENSEHAT"
+        (path "/e47212d5-bd6f-4bb8-9ec7-12aac08f34b5/e2c75964-4e94-4a3b-9ddf-38bb01f2971b"
+          (reference "J1") (unit 1)
+        )
+        (path "/e47212d5-bd6f-4bb8-9ec7-12aac08f34b5/8fedf9e5-f663-4f34-96fe-3613b2b14be8"
+          (reference "J3") (unit 1)
+        )
+      )
+    )
+  )
   (symbol (lib_id "power:GND") (at 270.51 132.08 0) (unit 1)
     (in_bom yes) (on_board yes) (dnp no) (fields_autoplaced)
@@
         )
       )
+    )
+  )
+  (symbol (lib_id "power:GND") (at 67.31 88.9 0) (unit 1)
+    (in_bom yes) (on_board yes) (dnp no) (fields_autoplaced)
+    (property "Reference" "#PWR040" (at 67.31 95.25 0)
+      (effects (font (size 1.27 1.27)) hide)
+    )
+    (property "Value" "GND" (at 67.31 93.98 0)
+      (effects (font (size 1.27 1.27)))
+    )
+    (property "Footprint" "" (at 67.31 88.9 0)
+      (effects (font (size 1.27 1.27)) hide)
+    )
+    (property "Datasheet" "" (at 67.31 88.9 0)
+      (effects (font (size 1.27 1.27)) hide)
+    )
+    (pin "1")
+    (instances
+      (project "STM32SENSEHAT"
+        (path "/e47212d5-bd6f-4bb8-9ec7-12aac08f34b5/8fedf9e5-f663-4f34-96fe-3613b2b14be8"
+          (reference "#PWR040") (unit 1)
+        )
+      )
